Commit message: update

File: interbotix_ros_xslocobots/interbotix_xslocobot_descriptions/urdf/arms/arm_control.urdf.xacro (robot description, xacro)
@@ -1,5 +1,6 @@
 <?xml version="1.0"?>
 <robot xmlns:xacro="http://ros.org/wiki/xacro">
-  <ros2_control name="XSHardwareInterface" type="system">
+  <!-- <ros2_control name="XSHardwareInterface" type="system"> -->
+  <ros2_control name="arm_controller" type="system">
     <hardware>
       <!-- If we are using the actual, physical robot -->
@@ -16,7 +17,9 @@
       </xacro:if>
       <!-- If simulating the robot in Gazebo Classic -->
-      <xacro:if value="${hardware_type == 'gz_classic'}">
+      <!-- <xacro:if value="${hardware_type == 'gz_classic'}">
         <plugin>gazebo_ros2_control/GazeboSystem</plugin>
-      </xacro:if>
+      </xacro:if> -->
+      <!-- bach-todo: add if -->
+      <plugin>gz_ros2_control/GazeboSimSystem</plugin>
     </hardware>
     <joint name="waist">

File: interbotix_ros_xslocobots/interbotix_xslocobot_descriptions/urdf/create3_version/wheel.urdf.xacro (robot description, xacro)
@@ -38,5 +38,5 @@
     <material>Gazebo/DarkGrey</material>
   </gazebo>
-  <xacro:if value="${hardware_type == 'gz_classic'}">
+  <!-- <xacro:if value="${hardware_type == 'gz_classic'}">
     <ros2_control name="${robot_name}/${wheel_link_name}_controller" type="system">
       <hardware>
@@ -49,5 +49,16 @@
       </joint>
     </ros2_control>
-  </xacro:if>
+  </xacro:if> -->
+  <!-- bach-todo: add if -->
+  <ros2_control name="GazeboSimSystem" type="system">
+    <hardware>
+      <plugin>gz_ros2_control/GazeboSimSystem</plugin>
+    </hardware>
+    <joint name="${wheel_joint_name}">
+      <state_interface name="velocity" />
+      <state_interface name="position" />
+      <command_interface name="velocity" />
+    </joint>
+  </ros2_control>
   <xacro:if value="${hardware_type == 'gz_ignition'}">
     <ros2_control name="${robot_name}/${wheel_link_name}_controller" type="system">

File: interbotix_ros_xslocobots/interbotix_xslocobot_descriptions/urdf/kobuki_version/locobot_kobuki.urdf.xacro (robot description, xacro)
@@ -104,5 +104,5 @@
       link="${robot_name}/wheel_left_link"/>
   </joint>
-  <xacro:if value="${hardware_type == 'gz_classic'}">
+  <!-- <xacro:if value="${hardware_type == 'gz_classic'}">
     <ros2_control name="wheel_left_joint_controller" type="system">
       <hardware>
@@ -115,5 +115,5 @@
       </joint>
     </ros2_control>
-  </xacro:if>
+  </xacro:if> -->
   <link name="${robot_name}/wheel_left_link">
     <visual>
@@ -131,4 +131,7 @@
           length="0.0206"
           radius="0.0352"/>
+        <!-- <cylinder
+          length="0.206"
+          radius="0.352"/> -->
       </geometry>
         <origin
@@ -140,4 +143,5 @@
         xyz="0 0 0"/>
       <mass value="0.01"/>
+      <!-- <mass value="0.0001"/> -->
       <inertia
         ixx="0.001"
@@ -167,5 +171,5 @@
       link="${robot_name}/wheel_right_link"/>
   </joint>
-  <xacro:if value="${hardware_type == 'gz_classic'}">
+  <!-- <xacro:if value="${hardware_type == 'gz_classic'}">
     <ros2_control name="wheel_right_joint_controller" type="system">
       <hardware>
@@ -178,5 +182,31 @@
       </joint>
     </ros2_control>
-  </xacro:if>
+  </xacro:if> -->
+  <!-- <ros2_control name="wheel_right_joint_controller" type="system">
+    <hardware>
+      <plugin>gazebo_ros2_control/GazeboSimSystem</plugin>
+    </hardware>
+    <joint name="wheel_right_joint">
+      <state_interface name="velocity" />
+      <state_interface name="position" />
+      <command_interface name="velocity" />
+    </joint>
+  </ros2_control> -->
+  <!-- bach-todo: add if -->
+  <ros2_control name="diffdrive_controller" type="system">
+    <hardware>
+      <plugin>gz_ros2_control/GazeboSimSystem</plugin>
+    </hardware>
+    <joint name="wheel_left_joint">
+      <state_interface name="velocity" />
+      <state_interface name="position" />
+      <command_interface name="velocity" />
+    </joint>
+    <joint name="wheel_right_joint">
+      <state_interface name="velocity" />
+      <state_interface name="position" />
+      <command_interface name="velocity" />
+    </joint>
+  </ros2_control>
   <link name="${robot_name}/wheel_right_link">
     <visual>
@@ -496,5 +526,5 @@
   <gazebo>
     <!-- Gazebo ROS Control -->
-    <xacro:if value="${hardware_type == 'gz_classic'}">
+    <!-- <xacro:if value="${hardware_type == 'gz_classic'}">
       <plugin name="gazebo_ros2_control" filename="libgazebo_ros2_control.so">
         <ros>
@@ -510,7 +540,16 @@
         <parameters> $(find interbotix_xslocobot_sim)/config/kobuki_version/$(arg robot_model)_controllers.yaml </parameters>
       </plugin>
-    </xacro:if>
+    </xacro:if> -->
+    <plugin filename="gz_ros2_control-system" name="gz_ros2_control::GazeboSimROS2ControlPlugin">
+      <ros>
+        <namespace>/$(arg robot_name)</namespace>
+      </ros>
+      <!-- <robot_param>robot_description</robot_param>
+      <robot_param_node>robot_state_publisher</robot_param_node> -->
+      <parameters>$(find interbotix_xslocobot_sim)/config/kobuki_version/$(arg robot_model)_controllers.yaml</parameters>
+      <!-- <controller_manager_name>controller_manager</controller_manager_name> -->
+    </plugin>
     <!-- Ground truth pose -->
-    <plugin filename="libgazebo_ros_p3d.so" name="p3d_base_controller">
+    <!-- <plugin filename="libgazebo_ros_p3d.so" name="p3d_base_controller">
       <ros>
         <remapping>odom:=sim_ground_truth_pose</remapping>
@@ -523,5 +562,10 @@
       <rpy_offset>0.0 0.0 0.0</rpy_offset>
       <gaussian_noise>0</gaussian_noise>
-    </plugin>
+    </plugin> -->
+    <!-- <plugin filename="libgz-sim-pose-publisher-system.so" name="gz::sim::systems::PosePublisher">
+        <publish_link_pose>true</publish_link_pose>
+        <publish_sensor_pose>true</publish_sensor_pose>
+        <use_world_frame>true</use_world_frame>
+    </plugin> -->
   </gazebo>
 </robot>

File: interbotix_ros_xslocobots/interbotix_xslocobot_descriptions/urdf/pan_and_tilt.urdf.xacro (robot description, xacro)
@@ -76,5 +76,5 @@
         damping="0.1"/>
     </joint>
-    <xacro:if value="${hardware_type == 'gz_classic'}">
+    <!-- <xacro:if value="${hardware_type == 'gz_classic'}">
       <ros2_control name="camera_controller" type="system">
         <hardware>
@@ -96,5 +96,25 @@
         </joint>
       </ros2_control>
-    </xacro:if>
+    </xacro:if> -->
+    <!-- bach-todo: add if -->
+    <ros2_control name="camera_controller" type="system">
+      <hardware>
+        <plugin>gz_ros2_control/GazeboSimSystem</plugin>
+      </hardware>
+      <joint name="pan">
+        <command_interface name="position">
+          <param name="min">"${-pi/2}"</param>
+          <param name="max">"${pi/2}"</param>
+        </command_interface>
+        <state_interface name="position"/>
+      </joint>
+      <joint name="tilt">
+        <command_interface name="position">
+          <param name="min">"${-pi/2}"</param>
+          <param name="max">"${radians(75)}"</param>
+        </command_interface>
+        <state_interface name="position"/>
+      </joint>
+    </ros2_control>
     <link name="${robot_name}/tilt_link">
       <visual>
@@ -202,5 +222,5 @@
       <origin rpy="0 0 0" xyz="0 0 0"/>
     </link>
-    <gazebo reference="camera_${robot_name}_link">
+    <!-- <gazebo reference="camera_${robot_name}_link">
       <sensor name="camera_frame_sensor" type="depth">
         <always_on>true</always_on>
@@ -244,4 +264,50 @@
         </plugin>
       </sensor>
+    </gazebo> -->
+    <gazebo reference="camera_${robot_name}_link">
+      <sensor name="camera_frame_sensor" type="depth">
+        <always_on>true</always_on>
+        <update_rate>30.0</update_rate>
+        <topic>/$(arg robot_name)/color/image_raw</topic>
+        <gz_frame_id>/$(arg robot_name)/camera_depth_link</gz_frame_id>
+        <camera>
+          <camera_info_topic>/$(arg robot_name)/color/camera_info</camera_info_topic>
+          <horizontal_fov>0.994837</horizontal_fov>
+          <image>
+            <format>R8G8B8</format>
+            <width>640</width>
+            <height>480</height>
+          </image>
+          <clip>
+            <near>0.01</near>
+            <far>10</far>
+          </clip>
+        </camera>
+        <!-- <plugin filename="libgazebo_ros_camera.so" name="camera_frame_controller"> -->
+          <!-- <ros>
+            <namespace>/$(arg robot_name)</namespace>
+          </ros> -->
+          <!-- <always_on>true</always_on> -->
+          <!-- <update_rate>0.0</update_rate> -->
+          <!-- <camera_name>camera</camera_name> -->
+          <!-- <image_topic_name>color/image_raw</image_topic_name> -->
+          <!-- <camera_info_topic_name>color/camera_info</camera_info_topic_name> -->
+          <!-- <depth_image_topic_name>aligned_depth_to_color/image_raw</depth_image_topic_name> -->
+          <!-- <depth_image_camera_info_topic_name>aligned_depth_to_color/camera_info</depth_image_camera_info_topic_name> -->
+          <!-- <point_cloud_topic_name>depth_registered/points</point_cloud_topic_name> -->
+          <!-- <frame_name>${robot_name}/camera_depth_link</frame_name> -->
+          <!-- <point_cloud_cutoff>0.01</point_cloud_cutoff>
+          <point_cloud_cutoff_max>10</point_cloud_cutoff_max>
+          <distortion_k1>0.00000001</distortion_k1>
+          <distortion_k2>0.00000001</distortion_k2>
+          <distortion_k3>0.00000001</distortion_k3>
+          <distortion_t1>0.00000001</distortion_t1>
+          <distortion_t2>0.00000001</distortion_t2>
+          <cx>0</cx>
+          <cy>0</cy>
+          <focal_length>0</focal_length>
+          <hack_baseline>0</hack_baseline> -->
+        <!-- </plugin> -->
+      </sensor>
     </gazebo>
   </xacro:macro>

Commit message: review: resolve comments

File: interbotix_ros_xslocobots/interbotix_xslocobot_descriptions/urdf/arms/arm_control.urdf.xacro (robot description, xacro)
@@ -1,6 +1,5 @@
 <?xml version="1.0"?>
 <robot xmlns:xacro="http://ros.org/wiki/xacro">
-  <!-- <ros2_control name="XSHardwareInterface" type="system"> -->
-  <ros2_control name="arm_controller" type="system">
+  <ros2_control name="XSHardwareInterface" type="system">
     <hardware>
       <!-- If we are using the actual, physical robot -->
@@ -16,10 +15,8 @@
         <plugin>fake_components/GenericSystem</plugin>
       </xacro:if>
-      <!-- If simulating the robot in Gazebo Classic -->
-      <!-- <xacro:if value="${hardware_type == 'gz_classic'}">
-        <plugin>gazebo_ros2_control/GazeboSystem</plugin>
-      </xacro:if> -->
-      <!-- bach-todo: add if -->
-      <plugin>gz_ros2_control/GazeboSimSystem</plugin>
+      <!-- If simulating the robot in Gazebo Sim -->
+      <xacro:if value="${hardware_type == 'gz_sim'}">
+        <plugin>gz_ros2_control/GazeboSimSystem</plugin>
+      </xacro:if>
     </hardware>
     <joint name="waist">

File: interbotix_ros_xslocobots/interbotix_xslocobot_descriptions/urdf/create3_version/wheel.urdf.xacro (robot description, xacro)
@@ -38,5 +38,5 @@
     <material>Gazebo/DarkGrey</material>
   </gazebo>
-  <!-- <xacro:if value="${hardware_type == 'gz_classic'}">
+  <xacro:if value="${hardware_type == 'gz_classic'}">
     <ros2_control name="${robot_name}/${wheel_link_name}_controller" type="system">
       <hardware>
@@ -49,16 +49,5 @@
       </joint>
     </ros2_control>
-  </xacro:if> -->
-  <!-- bach-todo: add if -->
-  <ros2_control name="GazeboSimSystem" type="system">
-    <hardware>
-      <plugin>gz_ros2_control/GazeboSimSystem</plugin>
-    </hardware>
-    <joint name="${wheel_joint_name}">
-      <state_interface name="velocity" />
-      <state_interface name="position" />
-      <command_interface name="velocity" />
-    </joint>
-  </ros2_control>
+  </xacro:if>
   <xacro:if value="${hardware_type == 'gz_ignition'}">
     <ros2_control name="${robot_name}/${wheel_link_name}_controller" type="system">

File: interbotix_ros_xslocobots/interbotix_xslocobot_descriptions/urdf/kobuki_version/locobot_kobuki.urdf.xacro (robot description, xacro)
@@ -104,16 +104,4 @@
       link="${robot_name}/wheel_left_link"/>
   </joint>
-  <!-- <xacro:if value="${hardware_type == 'gz_classic'}">
-    <ros2_control name="wheel_left_joint_controller" type="system">
-      <hardware>
-        <plugin>gazebo_ros2_control/GazeboSystem</plugin>
-      </hardware>
-      <joint name="wheel_left_joint">
-        <state_interface name="velocity" />
-        <state_interface name="position" />
-        <command_interface name="velocity" />
-      </joint>
-    </ros2_control>
-  </xacro:if> -->
   <link name="${robot_name}/wheel_left_link">
     <visual>
@@ -171,42 +159,4 @@
       link="${robot_name}/wheel_right_link"/>
   </joint>
-  <!-- <xacro:if value="${hardware_type == 'gz_classic'}">
-    <ros2_control name="wheel_right_joint_controller" type="system">
-      <hardware>
-        <plugin>gazebo_ros2_control/GazeboSystem</plugin>
-      </hardware>
-      <joint name="wheel_right_joint">
-        <state_interface name="velocity" />
-        <state_interface name="position" />
-        <command_interface name="velocity" />
-      </joint>
-    </ros2_control>
-  </xacro:if> -->
-  <!-- <ros2_control name="wheel_right_joint_controller" type="system">
-    <hardware>
-      <plugin>gazebo_ros2_control/GazeboSimSystem</plugin>
-    </hardware>
-    <joint name="wheel_right_joint">
-      <state_interface name="velocity" />
-      <state_interface name="position" />
-      <command_interface name="velocity" />
-    </joint>
-  </ros2_control> -->
-  <!-- bach-todo: add if -->
-  <ros2_control name="diffdrive_controller" type="system">
-    <hardware>
-      <plugin>gz_ros2_control/GazeboSimSystem</plugin>
-    </hardware>
-    <joint name="wheel_left_joint">
-      <state_interface name="velocity" />
-      <state_interface name="position" />
-      <command_interface name="velocity" />
-    </joint>
-    <joint name="wheel_right_joint">
-      <state_interface name="velocity" />
-      <state_interface name="position" />
-      <command_interface name="velocity" />
-    </joint>
-  </ros2_control>
   <link name="${robot_name}/wheel_right_link">
     <visual>
@@ -250,4 +200,21 @@
     <maxVel>1.0</maxVel>
   </gazebo>
+  <xacro:if value="${hardware_type == 'gz_sim'}">
+    <ros2_control name="diffdrive_controller" type="system">
+      <hardware>
+        <plugin>gz_ros2_control/GazeboSimSystem</plugin>
+      </hardware>
+      <joint name="wheel_left_joint">
+        <state_interface name="velocity" />
+        <state_interface name="position" />
+        <command_interface name="velocity" />
+      </joint>
+      <joint name="wheel_right_joint">
+        <state_interface name="velocity" />
+        <state_interface name="position" />
+        <command_interface name="velocity" />
+      </joint>
+    </ros2_control>
+  </xacro:if>
   <joint name="caster_front_joint" type="fixed">
     <origin
@@ -526,46 +493,25 @@
   <gazebo>
     <!-- Gazebo ROS Control -->
-    <!-- <xacro:if value="${hardware_type == 'gz_classic'}">
-      <plugin name="gazebo_ros2_control" filename="libgazebo_ros2_control.so">
-        <ros>
-          <namespace>/$(arg robot_name)</namespace>
-        </ros>
-        <robot_param>robot_description</robot_param>
-        <robot_param_node>robot_state_publisher</robot_param_node>
-        <parameters> $(find interbotix_xslocobot_sim)/config/kobuki_version/$(arg robot_model)_controllers.yaml </parameters>
-      </plugin>
-    </xacro:if>
     <xacro:if value="${hardware_type == 'gz_ignition'}">
       <plugin filename="ign_ros2_control-system" name="ign_ros2_control::IgnitionROS2ControlPlugin">
         <parameters> $(find interbotix_xslocobot_sim)/config/kobuki_version/$(arg robot_model)_controllers.yaml </parameters>
       </plugin>
-    </xacro:if> -->
-    <plugin filename="gz_ros2_control-system" name="gz_ros2_control::GazeboSimROS2ControlPlugin">
-      <ros>
-        <namespace>/$(arg robot_name)</namespace>
-      </ros>
-      <!-- <robot_param>robot_description</robot_param>
-      <robot_param_node>robot_state_publisher</robot_param_node> -->
-      <parameters>$(find interbotix_xslocobot_sim)/config/kobuki_version/$(arg robot_model)_controllers.yaml</parameters>
-      <!-- <controller_manager_name>controller_manager</controller_manager_name> -->
-    </plugin>
+    </xacro:if>
+    <xacro:if value="${hardware_type == 'gz_sim'}">
+      <plugin filename="gz_ros2_control-system" name="gz_ros2_control::GazeboSimROS2ControlPlugin">
+        <ros>
+          <namespace>/$(arg robot_name)</namespace>
+        </ros>
+        <parameters>$(find interbotix_xslocobot_sim)/config/kobuki_version/$(arg robot_model)_controllers.yaml</parameters>
+      </plugin>
+    </xacro:if>
     <!-- Ground truth pose -->
-    <!-- <plugin filename="libgazebo_ros_p3d.so" name="p3d_base_controller">
-      <ros>
-        <remapping>odom:=sim_ground_truth_pose</remapping>
-        <namespace>/$(arg robot_name)</namespace>
-      </ros>
-      <body_name>$(arg robot_name)/base_footprint</body_name>
-      <frame_name>world</frame_name>
-      <update_rate>100.0</update_rate>
-      <xyz_offset>0 0 0</xyz_offset>
-      <rpy_offset>0.0 0.0 0.0</rpy_offset>
-      <gaussian_noise>0</gaussian_noise>
-    </plugin> -->
-    <!-- <plugin filename="libgz-sim-pose-publisher-system.so" name="gz::sim::systems::PosePublisher">
-        <publish_link_pose>true</publish_link_pose>
-        <publish_sensor_pose>true</publish_sensor_pose>
-        <use_world_frame>true</use_world_frame>
-    </plugin> -->
+    <xacro:if value="${hardware_type == 'gz_sim'}">
+      <plugin filename="libgz-sim-pose-publisher-system.so" name="gz::sim::systems::PosePublisher">
+          <publish_link_pose>true</publish_link_pose>
+          <publish_sensor_pose>true</publish_sensor_pose>
+          <use_world_frame>true</use_world_frame>
+      </plugin>
+    </xacro:if>
   </gazebo>
 </robot>
