Commit message: update mobile_wx200.urdf.xacro: fix locobot twitching issue

File: interbotix_ros_xslocobots/interbotix_xslocobot_descriptions/urdf/arms/mobile_wx200.urdf.xacro (robot description, xacro)
@@ -86,6 +86,6 @@
       link="${robot_name}/shoulder_link"/>
     <dynamics
-      friction="0.1"
-      damping="0.1"/>
+      friction="0.2"
+      damping="1.5"/>
   </joint>
   <link name="${robot_name}/shoulder_link">
@@ -140,6 +140,6 @@
       link="${robot_name}/upper_arm_link"/>
     <dynamics
-      friction="0.1"
-      damping="0.1"/>
+      friction="0.2"
+      damping="1.5"/>
   </joint>
   <link name="${robot_name}/upper_arm_link">
@@ -194,6 +194,6 @@
       link="${robot_name}/forearm_link"/>
     <dynamics
-      friction="0.1"
-      damping="0.1"/>
+      friction="0.2"
+      damping="1.5"/>
   </joint>
   <link name="${robot_name}/forearm_link">
@@ -248,6 +248,6 @@
       link="${robot_name}/wrist_link"/>
     <dynamics
-      friction="0.1"
-      damping="0.1"/>
+      friction="0.2"
+      damping="1.5"/>
   </joint>
   <link name="${robot_name}/wrist_link">
@@ -304,6 +304,6 @@
         link="${robot_name}/gripper_link"/>
       <dynamics
-        friction="0.1"
-        damping="0.1"/>
+        friction="0.2"
+        damping="1.5"/>
     </joint>
     <link name="${robot_name}/gripper_link">
@@ -351,5 +351,5 @@
         link="${robot_name}/ee_arm_link"/>
     </joint>
-    <link name="${robot_name}/ee_arm_link">
+    <!-- <link name="${robot_name}/ee_arm_link">
       <inertial>
         <mass value="0.001"/>
@@ -362,5 +362,17 @@
           iyz="0"/>
       </inertial>
-    </link>
+    </link> -->
+    <link name="${robot_name}/ee_arm_link">
+    <inertial>
+      <mass value="0.05"/>
+      <inertia
+        ixx="0.00005"
+        iyy="0.00005"
+        izz="0.00005"
+        ixy="0"
+        ixz="0"
+        iyz="0"/>
+    </inertial>
+  </link>
     <joint name="gripper" type="continuous">
       <axis xyz="1 0 0"/>
@@ -376,6 +388,6 @@
         link="${robot_name}/gripper_prop_link"/>
       <dynamics
-        friction="0.1"
-        damping="0.1"/>
+        friction="0.2"
+        damping="1.5"/>
     </joint>
     <link name="${robot_name}/gripper_prop_link">
@@ -403,5 +415,5 @@
           rpy="0 0 ${pi/2}"
           xyz="0.0008460000 -0.0000016817 0.0000420000"/>
-        <mass value="0.00434"/>
+        <mass value="0.03"/>
         <inertia
           ixx="0.0000005923"
@@ -471,5 +483,5 @@
           link="${robot_name}/fingers_link"/>
       </joint>
-      <link name="${robot_name}/fingers_link">
+      <!-- <link name="${robot_name}/fingers_link">
         <inertial>
           <mass value="0.001"/>
@@ -482,5 +494,17 @@
             iyz="0"/>
         </inertial>
-      </link>
+      </link> -->
+      <link name="${robot_name}/fingers_link">
+      <inertial>
+        <mass value="0.03"/>
+        <inertia
+          ixx="0.00003"
+          iyy="0.00003"
+          izz="0.00003"
+          ixy="0"
+          ixz="0"
+          iyz="0"/>
+      </inertial>
+    </link>
       <!-- If the gripper fingers are being used, add those as well -->
       <xacro:if value="$(arg show_gripper_fingers)">
@@ -500,6 +524,6 @@
             link="${robot_name}/left_finger_link"/>
           <dynamics
-            friction="0.1"
-            damping="0.1"/>
+            friction="0.2"
+            damping="1.5"/>
         </joint>
         <link name="${robot_name}/left_finger_link">
@@ -554,6 +578,6 @@
             link="${robot_name}/right_finger_link"/>
           <dynamics
-            friction="0.1"
-            damping="0.1"/>
+            friction="0.2"
+            damping="1.5"/>
           <xacro:unless value="${hardware_type == 'gz_sim'}">
             <mimic
@@ -609,5 +633,5 @@
             link="${robot_name}/ee_gripper_link"/>
         </joint>
-        <link name="${robot_name}/ee_gripper_link">
+        <!-- <link name="${robot_name}/ee_gripper_link">
           <inertial>
             <mass value="0.001"/>
@@ -621,4 +645,17 @@
           </inertial>
         </link>
+         -->
+        <link name="${robot_name}/ee_gripper_link">
+        <inertial>
+          <mass value="0.02"/>
+          <inertia
+            ixx="0.00002"
+            iyy="0.00002"
+            izz="0.00002"
+            ixy="0"
+            ixz="0"
+            iyz="0"/>
+        </inertial>
+      </link>
       </xacro:if> <!-- show_gripper_fingers -->
     </xacro:if> <!-- show_gripper_bar -->
