Commit message: review: minor update

File: interbotix_ros_xslocobots/interbotix_xslocobot_descriptions/urdf/kobuki_version/locobot_kobuki.urdf.xacro (robot description, xacro)
@@ -119,7 +119,4 @@
           length="0.0206"
           radius="0.0352"/>
-        <!-- <cylinder
-          length="0.206"
-          radius="0.352"/> -->
       </geometry>
         <origin
@@ -131,5 +128,4 @@
         xyz="0 0 0"/>
       <mass value="0.01"/>
-      <!-- <mass value="0.0001"/> -->
       <inertia
         ixx="0.001"

File: interbotix_ros_xslocobots/interbotix_xslocobot_descriptions/urdf/pan_and_tilt.urdf.xacro (robot description, xacro)
@@ -76,8 +76,8 @@
         damping="0.1"/>
     </joint>
-    <!-- <xacro:if value="${hardware_type == 'gz_classic'}">
+    <xacro:if value="${hardware_type == 'gz_sim'}">
       <ros2_control name="camera_controller" type="system">
         <hardware>
-          <plugin>gazebo_ros2_control/GazeboSystem</plugin>
+          <plugin>gz_ros2_control/GazeboSimSystem</plugin>
         </hardware>
         <joint name="pan">
@@ -96,25 +96,5 @@
         </joint>
       </ros2_control>
-    </xacro:if> -->
-    <!-- bach-todo: add if -->
-    <ros2_control name="camera_controller" type="system">
-      <hardware>
-        <plugin>gz_ros2_control/GazeboSimSystem</plugin>
-      </hardware>
-      <joint name="pan">
-        <command_interface name="position">
-          <param name="min">"${-pi/2}"</param>
-          <param name="max">"${pi/2}"</param>
-        </command_interface>
-        <state_interface name="position"/>
-      </joint>
-      <joint name="tilt">
-        <command_interface name="position">
-          <param name="min">"${-pi/2}"</param>
-          <param name="max">"${radians(75)}"</param>
-        </command_interface>
-        <state_interface name="position"/>
-      </joint>
-    </ros2_control>
+    </xacro:if>
     <link name="${robot_name}/tilt_link">
       <visual>
@@ -222,47 +202,4 @@
       <origin rpy="0 0 0" xyz="0 0 0"/>
     </link>
-    <!-- <gazebo reference="camera_${robot_name}_link">
-      <sensor name="camera_frame_sensor" type="depth">
-        <always_on>true</always_on>
-        <update_rate>30.0</update_rate>
-        <camera>
-          <horizontal_fov>0.994837</horizontal_fov>
-          <image>
-            <format>R8G8B8</format>
-            <width>640</width>
-            <height>480</height>
-          </image>
-          <clip>
-            <near>0.01</near>
-            <far>10</far>
-          </clip>
-        </camera>
-        <plugin filename="libgazebo_ros_camera.so" name="camera_frame_controller">
-          <ros>
-            <namespace>/$(arg robot_name)</namespace>
-          </ros>
-          <always_on>true</always_on>
-          <update_rate>0.0</update_rate>
-          <camera_name>camera</camera_name>
-          <image_topic_name>color/image_raw</image_topic_name>
-          <camera_info_topic_name>color/camera_info</camera_info_topic_name>
-          <depth_image_topic_name>aligned_depth_to_color/image_raw</depth_image_topic_name>
-          <depth_image_camera_info_topic_name>aligned_depth_to_color/camera_info</depth_image_camera_info_topic_name>
-          <point_cloud_topic_name>depth_registered/points</point_cloud_topic_name>
-          <frame_name>${robot_name}/camera_depth_link</frame_name>
-          <point_cloud_cutoff>0.01</point_cloud_cutoff>
-          <point_cloud_cutoff_max>10</point_cloud_cutoff_max>
-          <distortion_k1>0.00000001</distortion_k1>
-          <distortion_k2>0.00000001</distortion_k2>
-          <distortion_k3>0.00000001</distortion_k3>
-          <distortion_t1>0.00000001</distortion_t1>
-          <distortion_t2>0.00000001</distortion_t2>
-          <cx>0</cx>
-          <cy>0</cy>
-          <focal_length>0</focal_length>
-          <hack_baseline>0</hack_baseline>
-        </plugin>
-      </sensor>
-    </gazebo> -->
     <gazebo reference="camera_${robot_name}_link">
       <sensor name="camera_frame_sensor" type="depth">
@@ -284,29 +221,4 @@
           </clip>
         </camera>
-        <!-- <plugin filename="libgazebo_ros_camera.so" name="camera_frame_controller"> -->
-          <!-- <ros>
-            <namespace>/$(arg robot_name)</namespace>
-          </ros> -->
-          <!-- <always_on>true</always_on> -->
-          <!-- <update_rate>0.0</update_rate> -->
-          <!-- <camera_name>camera</camera_name> -->
-          <!-- <image_topic_name>color/image_raw</image_topic_name> -->
-          <!-- <camera_info_topic_name>color/camera_info</camera_info_topic_name> -->
-          <!-- <depth_image_topic_name>aligned_depth_to_color/image_raw</depth_image_topic_name> -->
-          <!-- <depth_image_camera_info_topic_name>aligned_depth_to_color/camera_info</depth_image_camera_info_topic_name> -->
-          <!-- <point_cloud_topic_name>depth_registered/points</point_cloud_topic_name> -->
-          <!-- <frame_name>${robot_name}/camera_depth_link</frame_name> -->
-          <!-- <point_cloud_cutoff>0.01</point_cloud_cutoff>
-          <point_cloud_cutoff_max>10</point_cloud_cutoff_max>
-          <distortion_k1>0.00000001</distortion_k1>
-          <distortion_k2>0.00000001</distortion_k2>
-          <distortion_k3>0.00000001</distortion_k3>
-          <distortion_t1>0.00000001</distortion_t1>
-          <distortion_t2>0.00000001</distortion_t2>
-          <cx>0</cx>
-          <cy>0</cy>
-          <focal_length>0</focal_length>
-          <hack_baseline>0</hack_baseline> -->
-        <!-- </plugin> -->
       </sensor>
     </gazebo>

Commit message: update migration + replace PosePublisher with OdometryPublisher

File: interbotix_ros_xslocobots/interbotix_xslocobot_descriptions/urdf/kobuki_version/locobot_kobuki.urdf.xacro (robot description, xacro)
@@ -82,5 +82,5 @@
     </inertial>
   </link>
-  <gazebo reference="base_link">
+  <gazebo reference="${robot_name}/base_link">
     <mu1>0.3</mu1>
     <mu2>0.3</mu2>
@@ -90,5 +90,5 @@
       <visualize>true</visualize>
       <contact>
-        <collision>base_footprint</collision>
+        <collision>${robot_name}/base_footprint</collision>
       </contact>
     </sensor>
@@ -137,5 +137,5 @@
     </inertial>
   </link>
-  <gazebo reference="wheel_left_link">
+  <gazebo reference="${robot_name}/wheel_left_link">
     <mu1>1.0</mu1>
     <mu2>1.0</mu2>
@@ -188,5 +188,5 @@
     </inertial>
   </link>
-  <gazebo reference="wheel_right_link">
+  <gazebo reference="${robot_name}/wheel_right_link">
     <mu1>1.0</mu1>
     <mu2>1.0</mu2>
@@ -246,5 +246,5 @@
     </inertial>
   </link>
-  <gazebo reference="caster_front_link">
+  <gazebo reference="${robot_name}/caster_front_link">
     <mu1>0.0</mu1>
     <mu2>0.0</mu2>
@@ -287,5 +287,5 @@
     </inertial>
   </link>
-  <gazebo reference="caster_back_link">
+  <gazebo reference="${robot_name}/caster_back_link">
     <mu1>0.0</mu1>
     <mu2>0.0</mu2>
@@ -368,5 +368,5 @@
     </inertial>
   </link>
-  <gazebo reference="cliff_sensor_left_link">
+  <gazebo reference="${robot_name}/cliff_sensor_left_link">
     <sensor name="cliff_sensor_left" type="ray">
       <always_on>true</always_on>
@@ -415,5 +415,5 @@
     </inertial>
   </link>
-  <gazebo reference="cliff_sensor_right_link">
+  <gazebo reference="${robot_name}/cliff_sensor_right_link">
     <sensor name="cliff_sensor_right" type="ray">
       <always_on>true</always_on>
@@ -462,5 +462,5 @@
     </inertial>
   </link>
-  <gazebo reference="cliff_sensor_front_link">
+  <gazebo reference="${robot_name}/cliff_sensor_front_link">
     <sensor name="cliff_sensor_front" type="ray">
       <always_on>true</always_on>
@@ -504,10 +504,12 @@
       </plugin>
     </xacro:if>
-    <!-- Ground truth pose -->
+    <!-- Ground truth odometry -->
+    <!-- ref: https://github.com/dhanushshettigar/Getting-Started-With-ROS2/wiki/Differential-Drive-Robot-Teleop#2-include-the-vehicle-model-in-the-world-file -->
     <xacro:if value="${hardware_type == 'gz_sim'}">
-      <plugin filename="libgz-sim-pose-publisher-system.so" name="gz::sim::systems::PosePublisher">
-          <publish_link_pose>true</publish_link_pose>
-          <publish_sensor_pose>true</publish_sensor_pose>
-          <use_world_frame>true</use_world_frame>
+      <plugin
+        filename="gz-sim-odometry-publisher-system"
+        name="gz::sim::systems::OdometryPublisher">
+        <odom_frame>${robot_name}/base_footprint</odom_frame>
+        <robot_base_frame>${robot_name}/base_footprint</robot_base_frame>
       </plugin>
     </xacro:if>
